Commit message: sdfsdf

File: orient_description/fishbot/model.urdf.xacro (robot description, xacro)
@@ -202,5 +202,5 @@
         <child link="left_wheel" />
         <dynamics damping="0" friction="0" />
-        <limit effort="inf" velocity="inf" lower="-1e+16" upper="1e+16" />
+        <limit effort="5" velocity="10" lower="-100" upper="100" />
     </joint>
     <joint name="joint_tire_right" type="revolute">
@@ -210,5 +210,5 @@
         <child link="right_wheel" />
         <dynamics damping="0" friction="0" />
-        <limit effort="inf" velocity="inf" lower="-1e+16" upper="1e+16" />
+        <limit effort="5" velocity="10" lower="-100" upper="100" />
     </joint>
     <joint name="lidar_fixed_joint" type="fixed">

Commit message: sdfsdf

File: orient_description/fishbot/model.urdf.xacro (robot description, xacro)
@@ -155,5 +155,5 @@
             <origin xyz="0 0 0" rpy="0 -0 0" />
             <geometry>
-                <mesh filename="package://orient_description/fishbot/meshes/sensors/R2000.stl" scale="0.001 0.001 0.001" />
+                <mesh filename="package://orient_description/fishbot/meshes/sensors/R2000.dae" scale="0.001 0.001 0.001" />
             </geometry>
         </visual>
